File: USB2LT.kicad_sch (KiCad schematic)
At the start: 39 parts, among them J1 USB_B, J2 Mini-DIN-8, U1 FT230XS, U2 AZ1117H-ADJ, U3 TaskTalk-2.0, U4 SN65HVD11HD, U5 SN65HVD11HD

Commit message: New version
Parts:
- added D5: PWR, LED_SMD:LED_0805_2012Metric, symbol Device:LED
- added R13: 1K, Resistor_SMD:R_0805_2012Metric, symbol Device:R
- D1: value LED -> TX
- D2: value LED -> RX
- FB1: footprint Resistor_SMD:R_0402_1005Metric -> Resistor_SMD:R_0603_1608Metric
- J1: footprint Connector_USB:USB_B_TE_5787834_Vertical -> Connector_USB:UJ2-BH-1-TH_CUD
Connections:
- net +3.3V: now also R13.2
- net GND: now also D5.1 (K)
- net at U3.5 (CTS): now also U1.6 (~{CTS}); no longer U1.2 (~{RTS})
- new net: D5.2 (A), R13.1
Other:
- note added: "AMS1117-3.3 JLC# C6186"
- note added: "GZ1608D601TF 0603 JLC# C1002"
- title: (none) -> USB2LT

Commit message: Fix short
Connections:
- net GND: now also J2.4
Changed lines of the file:
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@@
   (junction (at 255.905 75.565) (diameter 0) (color 0 0 0 0)
   )
+  (junction (at 266.7 93.345) (diameter 0) (color 0 0 0 0)
+  )
   (junction (at 71.12 59.69) (diameter 0) (color 0 0 0 0)
   )
@@
     (stroke (width 0) (type default))
   )
+  (wire (pts (xy 266.7 93.345) (xy 266.7 97.79))
+    (stroke (width 0) (type default))
+  )
   (wire (pts (xy 71.12 57.15) (xy 71.12 59.69))
     (stroke (width 0) (type default))
@@
   )
   (wire (pts (xy 71.12 59.69) (xy 71.12 60.96))
+    (stroke (width 0) (type default))
+  )
+  (wire (pts (xy 266.7 93.218) (xy 266.7 93.345))
     (stroke (width 0) (type default))
   )
@@
         )
       )
+    )
+  )
+  (symbol (lib_id "power:GND") (at 266.7 97.79 0) (unit 1)
+    (in_bom yes) (on_board yes) (dnp no) (fields_autoplaced)
+    (property "Reference" "#PWR030" (at 266.7 104.14 0)
+      (effects (font (size 1.27 1.27)) hide)
+    )
+    (property "Value" "GND" (at 266.7 102.87 0)
+      (effects (font (size 1.27 1.27)))
+    )
+    (property "Footprint" "" (at 266.7 97.79 0)
+      (effects (font (size 1.27 1.27)) hide)
+    )
+    (property "Datasheet" "" (at 266.7 97.79 0)
+      (effects (font (size 1.27 1.27)) hide)
+    )
+    (pin "1")
+    (instances
+      (project "USB2LT"
+        (path "/b3c4ac27-577a-4ea6-b892-3c97e259bd60"
+          (reference "#PWR030") (unit 1)
+        )
+      )
