File: USB2LT.kicad_pcb (KiCad board)
At the start: 2 copper layers, 66.8 x 26.4 mm, 39 parts, among them J1 USB_B, J2 Mini-DIN-8, U1 FT230XS, U2 AZ1117H-ADJ, U3 TaskTalk-2.0, U4 SN65HVD11HD, U5 SN65HVD11HD

Commit message: New version
Parts:
- added D5: PWR, LED_SMD:LED_0805_2012Metric, F.Cu at (129.0, 86.1)
- added R13: 1K, Resistor_SMD:R_0805_2012Metric, F.Cu at (124.6, 86.1)
- D1: value LED -> TX
- D2: value LED -> RX
- FB1: footprint Resistor_SMD:R_0402_1005Metric -> Resistor_SMD:R_0603_1608Metric
- J1: footprint Connector_USB:USB_B_TE_5787834_Vertical -> Connector_USB:UJ2-BH-1-TH_CUD
- moved J1 9.15 mm to (119.7, 91.0), turned to -90 degrees
- moved FB1 2.79 mm to (124.3, 88.5)
- moved C6 2.79 mm to (129.0, 88.6)
Connections:
- U1 pad 2: Net-(U1-~{RTS}) -> unconnected-(U1-~{RTS}-Pad2)
- U1 pad 6: unconnected-(U1-~{CTS}-Pad6) -> Net-(U1-~{CTS})
- U3 pad 5: Net-(U1-~{RTS}) -> Net-(U1-~{CTS})
Routing:
- net Net-(U1-~{RTS}): track 15.6 -> 0.00 mm, vias 2 -> 0
- net Net-(U1-~{CTS}): track 0.00 -> 14.4 mm, vias 0 -> 2
- net +3.3V: track 126.3 -> 137.0 mm, vias 2 -> 3
- net Net-(J1-VBUS): track 22.3 -> 26.6 mm
- net Net-(U2-VI): track 33.8 -> 37.4 mm
- net Net-(D5-A): track 0.00 -> 2.55 mm
- net Net-(J1-D-): track 18.5 -> 20.7 mm
- net Net-(J1-D+): track 15.5 -> 14.1 mm
- net Net-(U1-CBUS2): track 9.48 -> 10.3 mm
- net GND: track 253.0 -> 253.7 mm
Other:
- board text added: "*"
- board text added: "LT2USB v2 RZ 2023"
- board text added: "LocalTalk to USB adapter RZ 2023 v. 2"
- board text removed: "LT2USB v1 RZ 2023"
- board text removed: "LocalTalk to USB adapter RZ 2023 v. 1"

Commit message: Fix short
Parts:
- added G***: LOGO, Symbol:cat, B.Cu at (154.7, 82.7)
Connections:
- J2 pad 4: unconnected-(J2-Pad4) -> GND
Routing:
- net Net-(J1-D-): track 20.7 -> 9.19 mm
- net GND: track 253.7 -> 263.8 mm

Commit message: v2.1
Other:
- board text added: "LT2USB v2.1 RZ 2024"
- board text added: "LocalTalk to USB adapter RZ 2024 v. 2.1"
- board text removed: "LT2USB v2 RZ 2023"
- board text removed: "LocalTalk to USB adapter RZ 2023 v. 2"
Changed lines of the file:
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@@
   (gr_rect (start 108.712 74.676) (end 175.514 101.092)
     (stroke (width 0.1) (type default)) (fill none) (layer "Edge.Cuts"))
-  (gr_text "LocalTalk to USB adapter\nRZ 2023\nv. 2" (at 164.211 97.663) (layer "B.Cu" knockout)
+  (gr_text "LocalTalk to USB adapter\nRZ 2024\nv. 2.1" (at 164.211 97.663) (layer "B.Cu" knockout)
     (effects (font (size 1 1) (thickness 0.15)) (justify left bottom mirror))
   )
-  (gr_text "LT2USB v2 RZ 2023" (at 140.208 100.203) (layer "F.SilkS")
+  (gr_text "LT2USB v2.1 RZ 2024" (at 140.208 100.203) (layer "F.SilkS")
     (effects (font (size 1 1) (thickness 0.15)) (justify left bottom))
   )
